File: Version 2/Kicad/MPU/MPU.kicad_sch (KiCad schematic)
At the start: 15 parts, among them U2 MPU-6050, U3 AP2112K-3.3

Commit message: Modified: Routing
Parts:
- removed C1: 4.7uF, Capacitor_SMD:CP_Elec_4x5.4, symbol Device:C
- removed C2, C6, C7: 0.1uF, Capacitor_SMD:CP_Elec_3x5.3, symbol Device:C
- removed C3, C5: 10uF, Capacitor_SMD:CP_Elec_3x5.3, symbol Device:C
- removed C4: 2.2uF, Capacitor_SMD:CP_Elec_3x5.3, symbol Device:C
- removed R1: 1k, Resistor_THT:R_Axial_DIN0204_L3.6mm_D1.6mm_P1.90mm_Vertical, symbol Device:R
- removed R2, R3: 4.7k, Resistor_THT:R_Axial_DIN0204_L3.6mm_D1.6mm_P1.90mm_Vertical, symbol Device:R
- removed R6: 4.7K, Resistor_THT:R_Axial_DIN0204_L3.6mm_D1.6mm_P1.90mm_Vertical, symbol Device:R
- removed U3: AP2112K-3.3, Package_TO_SOT_SMD:SOT-23-5, symbol Regulator_Linear:AP2112K-3.3
- added C1: 4.7uF, CL21A106KAYNNNE:CAPC2012X145N, symbol CL21A106KAYNNNE:CL21A106KAYNNNE
- added C10, C11, C9: 100nF, CL21A106KAYNNNE:CAPC2012X145N, symbol CL21A106KAYNNNE:CL21A106KAYNNNE
- added C2: 10uF, CL21A106KAYNNNE:CAPC2012X145N, symbol CL21A106KAYNNNE:CL21A106KAYNNNE
- added C8: 2.2uF, CL21A106KAYNNNE:CAPC2012X145N, symbol CL21A106KAYNNNE:CL21A106KAYNNNE
- added R5, R7, R8: 4.7k, 8-1879533-1:RESC1608X50N, symbol 8-1879533-1:8-1879533-1
- added R9: 1k, 8-1879533-1:RESC1608X50N, symbol 8-1879533-1:8-1879533-1
- added U1: AMS1117-3.3, Package_TO_SOT_SMD:SOT-223-3_TabPin2, symbol Regulator_Linear:AMS1117-3.3
- D2: footprint LED_THT:LED_D1.8mm_W1.8mm_H2.4mm_Horizontal_O1.27mm_Z8.2mm -> CL21A106KAYNNNE:CAPC2012X145N
Connections:
- net Earth is gone; now on net GND: D2.1 (K), U2.1 (CLKIN), U2.11 (FSYNC)
- net +3.3V: now also C10.2, C11.2, C2.2, R5.1, R7.1, R9.1, U1.2 (VO)
- net GND: now also C1.1, C10.1, C11.1, C2.1, C8.2, C9.1, R8.1, U1.1 (GND)
- net INT: now also PIN1.8 (Pin_8), U2.12 (INT)
- net SCL: now also R7.2
- net SDA: now also R5.2
- net VCC: now also C1.2, U1.3 (VI)
- net at PIN1.7 (Pin_7): now also R8.2
- net at U2.10 (REGOUT): now also C9.2
- net at U2.20 (CPOUT): now also C8.1
- net at D2.2 (A): now also R9.2
- net AD0: now reaches U2.9 (AD0)

Commit message: Modified: rerouting the pcb
Connections:
- net GND: now also PIN1.1 (Pin_1); no longer PIN1.2 (Pin_2)
- net VCC: now also PIN1.2 (Pin_2); no longer PIN1.1 (Pin_1)
Changed lines of the file:
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@@
     (stroke (width 0) (type default))
   )
-  (wire (pts (xy 222.25 93.98) (xy 232.41 93.98))
+  (wire (pts (xy 215.9 93.98) (xy 232.41 93.98))
     (stroke (width 0) (type default))
   )
@@
     (stroke (width 0) (type default))
   )
-  (wire (pts (xy 222.25 92.71) (xy 222.25 93.98))
+  (wire (pts (xy 215.9 91.44) (xy 215.9 93.98))
     (stroke (width 0) (type default))
   )
@@
     (stroke (width 0) (type default))
   )
+  (wire (pts (xy 207.01 95.25) (xy 207.01 96.52))
+    (stroke (width 0) (type default))
+  )
   (wire (pts (xy 119.38 45.72) (xy 119.38 59.69))
     (stroke (width 0) (type default))
@@
     (stroke (width 0) (type default))
   )
-  (wire (pts (xy 213.36 96.52) (xy 232.41 96.52))
+  (wire (pts (xy 207.01 96.52) (xy 232.41 96.52))
     (stroke (width 0) (type default))
   )
@@
     )
   )
-  (symbol (lib_id "power:VCC") (at 222.25 92.71 0) (unit 1)
-    (in_bom yes) (on_board yes) (dnp no) (fields_autoplaced)
-    (property "Reference" "#PWR015" (at 222.25 96.52 0)
-      (effects (font (size 1.27 1.27)) hide)
-    )
-    (property "Value" "VCC" (at 222.25 88.9 0)
-      (effects (font (size 1.27 1.27)))
-    )
-    (property "Footprint" "" (at 222.25 92.71 0)
-      (effects (font (size 1.27 1.27)) hide)
-    )
-    (property "Datasheet" "" (at 222.25 92.71 0)
-      (effects (font (size 1.27 1.27)) hide)
-    )
-    (pin "1")
-    (instances
-      (project "MPU"
-        (path "/e4ebcbfe-3eac-4fb9-9225-5f736cfefaf3"
-          (reference "#PWR015") (unit 1)
-        )
-      )
-    )
-  )
   (symbol (lib_id "power:GND") (at 190.5 49.53 0) (unit 1)
     (in_bom yes) (on_board yes) (dnp no) (fields_autoplaced)
@@
     )
   )
+  (symbol (lib_id "power:GND") (at 215.9 91.44 180) (unit 1)
+    (in_bom yes) (on_board yes) (dnp no) (fields_autoplaced)
+    (property "Reference" "#PWR01" (at 215.9 85.09 0)
+      (effects (font (size 1.27 1.27)) hide)
+    )
+    (property "Value" "GND" (at 215.9 87.63 0)
+      (effects (font (size 1.27 1.27)))
+    )
+    (property "Footprint" "" (at 215.9 91.44 0)
+      (effects (font (size 1.27 1.27)) hide)
+    )
+    (property "Datasheet" "" (at 215.9 91.44 0)
+      (effects (font (size 1.27 1.27)) hide)
+    )
+    (pin "1")
+    (instances
+      (project "MPU"
+        (path "/e4ebcbfe-3eac-4fb9-9225-5f736cfefaf3"
+          (reference "#PWR01") (unit 1)
+        )
+      )
+    )
+  )
   (symbol (lib_id "power:GND") (at 172.72 97.79 90) (unit 1)
     (in_bom yes) (on_board yes) (dnp no) (fields_autoplaced)
@@
     )
   )
+  (symbol (lib_id "power:VCC") (at 207.01 95.25 0) (unit 1)
+    (in_bom yes) (on_board yes) (dnp no)
+    (property "Reference" "#PWR03" (at 207.01 99.06 0)
+      (effects (font (size 1.27 1.27)) hide)
+    )
+    (property "Value" "VCC" (at 207.01 91.44 0)
+      (effects (font (size 1.27 1.27)))
+    )
+    (property "Footprint" "" (at 207.01 95.25 0)
+      (effects (font (size 1.27 1.27)) hide)
+    )
+    (property "Datasheet" "" (at 207.01 95.25 0)
+      (effects (font (size 1.27 1.27)) hide)
+    )
+    (pin "1")
+    (instances
+      (project "MPU"
+        (path "/e4ebcbfe-3eac-4fb9-9225-5f736cfefaf3"
+          (reference "#PWR03") (unit 1)
+        )
+      )
+    )
+  )
   (symbol (lib_id "8-1879533-1:8-1879533-1") (at 267.97 26.67 0) (unit 1)
     (in_bom yes) (on_board yes) (dnp no) (fields_autoplaced)
@@
         )
       )
-    )
-  )
-  (symbol (lib_id "power:GND") (at 213.36 96.52 270) (unit 1)
-    (in_bom yes) (on_board yes) (dnp no) (fields_autoplaced)
-    (property "Reference" "#PWR01" (at 207.01 96.52 0)
-      (effects (font (size 1.27 1.27)) hide)
-    )
-    (property "Value" "GND" (at 209.55 97.155 90)
-      (effects (font (size 1.27 1.27)) (justify right))
-    )
-    (property "Footprint" "" (at 213.36 96.52 0)
-      (effects (font (size 1.27 1.27)) hide)
-    )
-    (property "Datasheet" "" (at 213.36 96.52 0)
-      (effects (font (size 1.27 1.27)) hide)
-    )
-    (pin "1")
-    (instances
-      (project "MPU"
-        (path "/e4ebcbfe-3eac-4fb9-9225-5f736cfefaf3"
-          (reference "#PWR01") (unit 1)
-        )
-      )
